Commit message: updated urdf positions

File: jo_description/urdf/D455.xacro (robot description, xacro)
@@ -2,10 +2,10 @@
 <robot xmlns:xacro="http://ros.org/wiki/xacro">
     <xacro:property name="PI" value="3.141592" />
-    <xacro:property name="b2c_x" value="1.0" />
-    <xacro:property name="b2c_y" value="0.0" />
-    <xacro:property name="b2c_z" value="0.0" />
+    <xacro:property name="b2c_x" value="-0.30639" />
+    <xacro:property name="b2c_y" value="0.01414" />
+    <xacro:property name="b2c_z" value="0.27801" />
     <xacro:property name="b2c_R" value="0.0" />
     <xacro:property name="b2c_P" value="0.0" />
-    <xacro:property name="b2c_Y" value="0.0" />
+    <xacro:property name="b2c_Y" value="${PI}" />
     <xacro:property name="camera_mass" value="0.125" />
     <xacro:property name="camera_len_rad" value="0.0508" />
@@ -26,5 +26,5 @@
             </collision>
             <visual>
-                <origin xyz="0 0 0" rpy="0 0 0"/>
+                <origin xyz="0 0 0" rpy="0 ${PI/2} 0"/>
                 <geometry>
                     <cylinder radius="${camera_len_rad}" length="${camera_len_h}"/>

File: jo_description/urdf/imu.xacro (robot description, xacro)
@@ -2,7 +2,7 @@
 <robot xmlns:xacro="http://ros.org/wiki/xacro">
     <xacro:property name="PI" value="3.141592" />
-    <xacro:property name="b2i_x" value="0.0" />
-    <xacro:property name="b2i_y" value="0.0" />
-    <xacro:property name="b2i_z" value="0.0" />
+    <xacro:property name="b2i_x" value="0.22172" />
+    <xacro:property name="b2i_y" value="0.02606" />
+    <xacro:property name="b2i_z" value="0.28202" />
     <xacro:property name="b2i_R" value="0.0" />
     <xacro:property name="b2i_P" value="0.0" />

File: jo_description/urdf/robot_core.xacro (robot description, xacro)
@@ -28,4 +28,7 @@
         <color rgba="0 0 0 1"/>
     </material>
+    <material name="black_t">
+        <color rgba="0 0 0 0.5"/>
+    </material>
     <material name="red">
         <color rgba="1 0 0 1"/>
@@ -175,3 +178,26 @@
         <mu2 value="0.001"/>
     </gazebo>
+    <link name="rack">
+        <visual>
+            <origin xyz=" 0 0 0"/>
+            <geometry>
+                <box size="0.6 0.37 0.47"/>
+            </geometry>
+            <material name="black_t"/>
+        </visual>
+        <collision>
+            <origin xyz="0 0 0"/>
+            <geometry>
+                <box size="${chassis_length*0.6} ${chassis_width*0.8} 0.5"/>
+            </geometry>
+        </collision>
+        <xacro:inertial_box mass="0.1" x="${chassis_length*0.6}" y="${chassis_width*0.8}" z="0.5">
+            <origin xyz="0 0 0" rpy="0 0 0"/>
+        </xacro:inertial_box>
+    </link>
+    <joint name="base2rack" type="fixed">
+        <parent link="base_link"/>
+        <child link="rack"/>
+        <origin xyz="0.02 0 0.25"/>
+    </joint>
 </robot>

File: jo_description/urdf/velodyne.xacro (robot description, xacro)
@@ -2,7 +2,7 @@
 <robot xmlns:xacro="http://ros.org/wiki/xacro">
     <xacro:property name="PI" value="3.141592" />
-    <xacro:property name="b2l_x" value="0.0" />
-    <xacro:property name="b2l_y" value="0.0" />
-    <xacro:property name="b2l_z" value="0.2" />
+    <xacro:property name="b2l_x" value="0.03" />
+    <xacro:property name="b2l_y" value="0.0286" />
+    <xacro:property name="b2l_z" value="0.630" />
     <xacro:property name="b2l_R" value="0.0" />
     <xacro:property name="b2l_P" value="0.0" />
