Commit message: added rviz configs; fixed some values in the urdf

File: jo_description/urdf/imu.xacro (robot description, xacro)
@@ -39,5 +39,5 @@
                     <gz_frame_id>imu_link</gz_frame_id>
                     <always_on>1</always_on>
-                    <update_rate>100</update_rate>
+                    <update_rate>200</update_rate>
                     <visualize>true</visualize>
                     <topic>imu</topic>

File: jo_description/urdf/velodyne.xacro (robot description, xacro)
@@ -9,6 +9,6 @@
     <xacro:property name="b2l_Y" value="0.0" />
     <xacro:property name="lidar_mass" value="0.125" />
-    <xacro:property name="lidar_len_rad" value="0.0508" />
-    <xacro:property name="lidar_len_h" value="0.055" />
+    <xacro:property name="lidar_len_rad" value="0.07" />
+    <xacro:property name="lidar_len_h" value="0.072" />
     <xacro:include filename="$(find jo_description)/urdf/inertial_macros.xacro" />
     <xacro:macro name="lidar_sensor" params="namespace">
