Commit message: Scale up turtlebot dimensions
- Body: 0.6x0.6x1.1m (top at ~1.22m from ground)
- Wheels: radius 0.12m, separation 0.76m
- Caster repositioned to match new ground clearance
- Inertia updated accordingly

Co-Authored-By: Claude Sonnet 4.6 <noreply@anthropic.com>

File: turtlebot_description/urdf/turtlebot.urdf (robot description, URDF)
Before this commit: robot turtlebot, 5 links, 4 joints
Links:
- link base_link: mass 8.2573504e-01 -> 20.0; geometry collision box size=0.6 0.6 1.1; visual box size=0.6 0.6 1.1
- link caster_back_link: mass 0.005 -> 0.05; geometry collision sphere radius=0.02
- link wheel_left_link: mass 2.8498940e-02 -> 0.5; geometry collision cylinder length=0.06 radius=0.12; visual cylinder length=0.06 radius=0.12
- link wheel_right_link: mass 2.8498940e-02 -> 0.5; geometry collision cylinder length=0.06 radius=0.12; visual cylinder length=0.06 radius=0.12
Joints:
- joint base_joint: origin xyz=0.0 0.0 0.010 rpy=0 0 0 -> xyz=0.0 0.0 0.12 rpy=0 0 0
- joint caster_back_joint: origin xyz=-0.081 0 -0.004 rpy=-1.57 0 0 -> xyz=-0.28 0 -0.10 rpy=0 0 0
- joint wheel_left_joint: origin xyz=0.0 0.08 0.023 rpy=-1.57 0 0 -> xyz=0.0 0.38 0.0 rpy=-1.57 0 0
- joint wheel_right_joint: origin xyz=0.0 -0.08 0.023 rpy=-1.57 0 0 -> xyz=0.0 -0.38 0.0 rpy=-1.57 0 0

Commit message: turtlebot: add two front passive wheels for pitch stability
Two non-steering continuous-joint wheels at x=+0.28, y=±0.20.
Same radius as drive wheels (0.12m) so they contact the ground at the
same level. Extends the support polygon forward and prevents the robot
from tipping when decelerating.

Co-Authored-By: Claude Sonnet 4.6 <noreply@anthropic.com>

File: turtlebot_description/urdf/turtlebot.urdf (robot description, URDF)
Before this commit: robot turtlebot, 5 links, 4 joints
Links:
- added link wheel_front_left_link, mass 0.1; collision cylinder length=0.04 radius=0.12; visual cylinder length=0.04 radius=0.12
- added link wheel_front_right_link, mass 0.1; collision cylinder length=0.04 radius=0.12; visual cylinder length=0.04 radius=0.12
Joints:
- added joint wheel_front_left_joint: type continuous, parent base_link, child wheel_front_left_link, origin xyz=0.28 0.20 0.0 rpy=-1.57 0 0, axis 0 0 1
- added joint wheel_front_right_joint: type continuous, parent base_link, child wheel_front_right_link, origin xyz=0.28 -0.20 0.0 rpy=-1.57 0 0, axis 0 0 1
